Commit message: updated test for jointmodifier

File: tests/test_model.urdf (robot description, URDF)
Before this commit: robot test_model, 6 links, 5 joints
Joints:
- joint joint_to_ground: origin xyz=0 0 0.5 -> xyz=0 0 0

Commit message: improved test model to be more useful for tests

File: tests/test_model.urdf (robot description, URDF)
Before this commit: robot test_model, 6 links, 5 joints
Links:
- link aligned_link: geometry collision cylinder length=2 radius=0.2; visual cylinder length=2 radius=0.2
- link base_link: geometry collision sphere radius=0.5; visual sphere radius=0.5
- link connector_link_1: geometry collision sphere radius=0.5; visual sphere radius=0.5
- link non_aligned_link: geometry collision box size=0.4 0.4 2; visual box size=0.4 0.4 2
Joints:
- joint aligned_link_joint_after: origin xyz=0 0 1.5 -> xyz=0 0 2
- joint aligned_link_joint_before: origin xyz=0 0 1.5 -> xyz=0 0 0
- joint non_aligned_link_joint_after: origin xyz=0 0 1.3 -> xyz=0 0 2
- joint non_aligned_link_joint_before: origin xyz=0.2 0.2 1.7 -> (none)

Commit message: updated test model to have non-zero values in origin of one joint

File: tests/test_model.urdf (robot description, URDF)
Before this commit: robot test_model, 6 links, 5 joints
Joints:
- joint non_aligned_link_joint_after: origin xyz=0 0 2 -> xyz=0.5 0.5 2

Commit message: updated test_model to reflect more test cases

File: tests/test_model.urdf (robot description, URDF)
Before this commit: robot test_model, 6 links, 5 joints
Links:
- removed link world
Joints:
- removed joint joint_to_ground
- joint aligned_link_joint_after: origin xyz=0 0 2 -> xyz=0 0 3
- joint non_aligned_link_joint_after: origin xyz=0.5 0.5 2 -> xyz=0 0 2
